Commit message: refactor: consolidate CAD and collision models

File: model/collision/ur10_cell.collision.xacro (robot description, xacro)
@@ -67,10 +67,10 @@
   <link name="$(arg tf_prefix)ft_mount_plate">
     <visual>
-      <origin xyz="0 0 $(PLATE_D/2)" rpy="0 0 0"/>
+      <origin xyz="0 0 ${PLATE_D/2}" rpy="0 0 0"/>
       <geometry><cylinder radius="0.045" length="${PLATE_D}"/></geometry>
       <material name="finger_metal"/>
     </visual>
     <collision>
-      <origin xyz="0 0 $(PLATE_D/2)" rpy="0 0 0"/>
+      <origin xyz="0 0 ${PLATE_D/2}" rpy="0 0 0"/>
       <geometry><cylinder radius="0.045" length="${PLATE_D}"/></geometry>
     </collision>
@@ -88,10 +88,10 @@
   <link name="$(arg tf_prefix)ati_sensor">
     <visual>
-      <origin xyz="0 0 $(PLATE_D + FT_D/2)" rpy="0 0 0"/>
+      <origin xyz="0 0 ${PLATE_D + FT_D/2}" rpy="0 0 0"/>
       <geometry><cylinder radius="${FT_R}" length="${FT_D}"/></geometry>
       <material name="ati_blue"/>
     </visual>
     <collision>
-      <origin xyz="0 0 $(PLATE_D + FT_D/2)" rpy="0 0 0"/>
+      <origin xyz="0 0 ${PLATE_D + FT_D/2}" rpy="0 0 0"/>
       <geometry><cylinder radius="${FT_R}" length="${FT_D}"/></geometry>
     </collision>
@@ -100,15 +100,15 @@
     <parent link="$(arg tf_prefix)ft_mount_plate"/>
     <child link="$(arg tf_prefix)ati_sensor"/>
-    <origin xyz="0 0 $(PLATE_D)" rpy="0 0 0"/>
+    <origin xyz="0 0 ${PLATE_D}" rpy="0 0 0"/>
   </joint>
   <!-- ============ 3. 传感器 → 夹爪 耦合板 ============ -->
   <link name="$(arg tf_prefix)gripper_coupling">
     <visual>
-      <origin xyz="0 0 $(PLATE_D + FT_D + PLATE_D/2)" rpy="0 0 0"/>
+      <origin xyz="0 0 ${PLATE_D + FT_D + PLATE_D/2}" rpy="0 0 0"/>
       <geometry><cylinder radius="0.0364" length="${PLATE_D}"/></geometry>
       <material name="finger_metal"/>
     </visual>
     <collision>
-      <origin xyz="0 0 $(PLATE_D + FT_D + PLATE_D/2)" rpy="0 0 0"/>
+      <origin xyz="0 0 ${PLATE_D + FT_D + PLATE_D/2}" rpy="0 0 0"/>
       <geometry><cylinder radius="0.0364" length="${PLATE_D}"/></geometry>
     </collision>
@@ -117,5 +117,5 @@
     <parent link="$(arg tf_prefix)ati_sensor"/>
     <child link="$(arg tf_prefix)gripper_coupling"/>
-    <origin xyz="0 0 $(PLATE_D + FT_D)" rpy="0 0 0"/>
+    <origin xyz="0 0 ${PLATE_D + FT_D}" rpy="0 0 0"/>
   </joint>
   <!-- ============ 4. Robotiq 2F-85 夹爪主体 ============ -->
@@ -124,11 +124,11 @@
   <link name="$(arg tf_prefix)gripper_base">
     <visual>
-      <origin xyz="0 0 $(2*PLATE_D + FT_D + GRIP_D/2)" rpy="0 0 0"/>
-      <geometry><box size="0.1435 $(GRIP_W) $(GRIP_D)"/></geometry>
+      <origin xyz="0 0 ${2*PLATE_D + FT_D + GRIP_D/2}" rpy="0 0 0"/>
+      <geometry><box size="0.1435 ${GRIP_W} ${GRIP_D}"/></geometry>
       <material name="gripper_gray"/>
     </visual>
     <collision>
-      <origin xyz="0 0 $(2*PLATE_D + FT_D + GRIP_D/2)" rpy="0 0 0"/>
-      <geometry><box size="0.1435 $(GRIP_W) $(GRIP_D)"/></geometry>
+      <origin xyz="0 0 ${2*PLATE_D + FT_D + GRIP_D/2}" rpy="0 0 0"/>
+      <geometry><box size="0.1435 ${GRIP_W} ${GRIP_D}"/></geometry>
     </collision>
   </link>
@@ -136,5 +136,5 @@
     <parent link="$(arg tf_prefix)gripper_coupling"/>
     <child link="$(arg tf_prefix)gripper_base"/>
-    <origin xyz="0 0 $(2*PLATE_D + FT_D)" rpy="0 0 0"/>
+    <origin xyz="0 0 ${2*PLATE_D + FT_D}" rpy="0 0 0"/>
   </joint>
   <!-- ============ 5. 左右手指（prismatic） ============ -->
@@ -144,11 +144,11 @@
   <link name="$(arg tf_prefix)left_finger">
     <visual>
-      <origin xyz="0 0 $(2*PLATE_D + FT_D + GRIP_D + FING_L/2)" rpy="0 0 0"/>
-      <geometry><box size="0.018 0.022 $(FING_L)"/></geometry>
-      <material name="finger_metal"/>
-    </visual>
-    <collision>
-      <origin xyz="0 0 $(2*PLATE_D + FT_D + GRIP_D + FING_L/2)" rpy="0 0 0"/>
-      <geometry><box size="0.018 0.022 $(FING_L)"/></geometry>
+      <origin xyz="0 0 ${2*PLATE_D + FT_D + GRIP_D + FING_L/2}" rpy="0 0 0"/>
+      <geometry><box size="0.018 0.022 ${FING_L}"/></geometry>
+      <material name="finger_metal"/>
+    </visual>
+    <collision>
+      <origin xyz="0 0 ${2*PLATE_D + FT_D + GRIP_D + FING_L/2}" rpy="0 0 0"/>
+      <geometry><box size="0.018 0.022 ${FING_L}"/></geometry>
     </collision>
   </link>
@@ -156,5 +156,5 @@
     <parent link="$(arg tf_prefix)gripper_base"/>
     <child link="$(arg tf_prefix)left_finger"/>
-    <origin xyz="0.0313 0 $(2*PLATE_D + FT_D + GRIP_D)" rpy="0 0 0"/>
+    <origin xyz="0.0313 0 ${2*PLATE_D + FT_D + GRIP_D}" rpy="0 0 0"/>
     <axis xyz="1 0 0"/>
     <limit lower="0" upper="0.0425" effort="100" velocity="0.15"/>
@@ -162,11 +162,11 @@
   <link name="$(arg tf_prefix)right_finger">
     <visual>
-      <origin xyz="0 0 $(2*PLATE_D + FT_D + GRIP_D + FING_L/2)" rpy="0 0 0"/>
-      <geometry><box size="0.018 0.022 $(FING_L)"/></geometry>
-      <material name="finger_metal"/>
-    </visual>
-    <collision>
-      <origin xyz="0 0 $(2*PLATE_D + FT_D + GRIP_D + FING_L/2)" rpy="0 0 0"/>
-      <geometry><box size="0.018 0.022 $(FING_L)"/></geometry>
+      <origin xyz="0 0 ${2*PLATE_D + FT_D + GRIP_D + FING_L/2}" rpy="0 0 0"/>
+      <geometry><box size="0.018 0.022 ${FING_L}"/></geometry>
+      <material name="finger_metal"/>
+    </visual>
+    <collision>
+      <origin xyz="0 0 ${2*PLATE_D + FT_D + GRIP_D + FING_L/2}" rpy="0 0 0"/>
+      <geometry><box size="0.018 0.022 ${FING_L}"/></geometry>
     </collision>
   </link>
@@ -174,5 +174,5 @@
     <parent link="$(arg tf_prefix)gripper_base"/>
     <child link="$(arg tf_prefix)right_finger"/>
-    <origin xyz="-0.0313 0 $(2*PLATE_D + FT_D + GRIP_D)" rpy="0 0 0"/>
+    <origin xyz="-0.0313 0 ${2*PLATE_D + FT_D + GRIP_D}" rpy="0 0 0"/>
     <axis xyz="-1 0 0"/>
     <limit lower="0" upper="0.0425" effort="100" velocity="0.15"/>
@@ -185,10 +185,10 @@
   <link name="$(arg tf_prefix)camera_link">
     <visual>
-      <origin xyz="$(CAM_X) $(CAM_Y) $(CAM_Z)" rpy="0 0 0"/>
+      <origin xyz="${CAM_X} ${CAM_Y} ${CAM_Z}" rpy="0 0 0"/>
       <geometry><box size="0.160 0.1365 0.195"/></geometry>
       <material name="camera_dark"/>
     </visual>
     <collision>
-      <origin xyz="$(CAM_X) $(CAM_Y) $(CAM_Z)" rpy="0 0 0"/>
+      <origin xyz="${CAM_X} ${CAM_Y} ${CAM_Z}" rpy="0 0 0"/>
       <geometry><box size="0.160 0.1365 0.195"/></geometry>
     </collision>
